Commit message: New URDF With Labels
1 - bottom; 2 - middle; 3 - top
BL - Back-Left
FR - Front-Right

File: ROS_Stack/src/zeta_description/urdf/zeta.xacro (robot description, xacro)
@@ -3,7 +3,5 @@
 <xacro:include filename="$(find zeta_description)/urdf/materials.xacro" />
 <xacro:include filename="$(find zeta_description)/urdf/zeta.trans" />
-<xacro:include filename="$(find zeta_description)/gazebo/zeta_materials.gazebo" />
-<xacro:include filename="$(find zeta_description)/gazebo/zeta_physics.gazebo" />
-<xacro:include filename="$(find zeta_description)/gazebo/zeta_plugins.gazebo" />
+<xacro:include filename="$(find zeta_description)/urdf/zeta.gazebo" />
 <link name="base_link">
   <inertial>
@@ -306,5 +304,5 @@
   </collision>
 </link>
-<joint name="Rev46" type="continuous">
+<joint name="BL_1" type="continuous">
   <origin rpy="0 0 0" xyz="-0.054447 0.0 -0.054447"/>
   <parent link="BL_motor_block_1"/>
@@ -312,5 +310,5 @@
   <axis xyz="0.0 1.0 -0.0"/>
 </joint>
-<joint name="Rev47" type="continuous">
+<joint name="BL_2" type="continuous">
   <origin rpy="0 0 0" xyz="0.0164 0.075469 -0.051319"/>
   <parent link="BL_top_1"/>
@@ -318,5 +316,5 @@
   <axis xyz="0.0 -1.0 0.0"/>
 </joint>
-<joint name="Rev48" type="continuous">
+<joint name="BL_3" type="continuous">
   <origin rpy="0 0 0" xyz="-0.295505 0.128052 0.206491"/>
   <parent link="base_link"/>
@@ -324,5 +322,5 @@
   <axis xyz="1.0 -0.0 -0.0"/>
 </joint>
-<joint name="Rev49" type="continuous">
+<joint name="BR_1" type="continuous">
   <origin rpy="0 0 0" xyz="-0.054447 0.0 -0.054447"/>
   <parent link="BR_motor_block_1"/>
@@ -330,5 +328,5 @@
   <axis xyz="-0.0 -1.0 0.0"/>
 </joint>
-<joint name="Rev50" type="continuous">
+<joint name="BR_2" type="continuous">
   <origin rpy="0 0 0" xyz="0.0164 -0.075469 -0.051319"/>
   <parent link="BR_top_1"/>
@@ -336,5 +334,5 @@
   <axis xyz="-0.0 -1.0 0.0"/>
 </joint>
-<joint name="Rev51" type="continuous">
+<joint name="BR_3" type="continuous">
   <origin rpy="0 0 0" xyz="-0.295505 0.048652 0.206491"/>
   <parent link="base_link"/>
@@ -342,5 +340,5 @@
   <axis xyz="-1.0 0.0 0.0"/>
 </joint>
-<joint name="Rev54" type="continuous">
+<joint name="FR_3" type="continuous">
   <origin rpy="0 0 0" xyz="-0.024505 0.048652 0.206491"/>
   <parent link="base_link"/>
@@ -348,5 +346,5 @@
   <axis xyz="-1.0 0.0 0.0"/>
 </joint>
-<joint name="Rev55" type="continuous">
+<joint name="FL_1" type="continuous">
   <origin rpy="0 0 0" xyz="-0.054447 0.0 -0.054447"/>
   <parent link="FL_motor_block_1"/>
@@ -354,5 +352,5 @@
   <axis xyz="0.0 -1.0 -0.0"/>
 </joint>
-<joint name="Rev56" type="continuous">
+<joint name="FL_2" type="continuous">
   <origin rpy="0 0 0" xyz="0.0164 0.075469 -0.051319"/>
   <parent link="FL_top_1"/>
@@ -360,5 +358,5 @@
   <axis xyz="0.0 -1.0 0.0"/>
 </joint>
-<joint name="Rev57" type="continuous">
+<joint name="FL_3" type="continuous">
   <origin rpy="0 0 0" xyz="-0.024505 0.128052 0.206491"/>
   <parent link="base_link"/>
@@ -366,15 +364,15 @@
   <axis xyz="1.0 -0.0 -0.0"/>
 </joint>
-<joint name="Rigid58" type="fixed">
+<joint name="R_Pipe" type="fixed">
   <origin rpy="0 0 0" xyz="-0.260605 0.067967 0.206491"/>
   <parent link="base_link"/>
   <child link="R_Pipe_1"/>
 </joint>
-<joint name="Rigid59" type="fixed">
+<joint name="L_Pipe" type="fixed">
   <origin rpy="0 0 0" xyz="-0.260605 0.108737 0.206491"/>
   <parent link="base_link"/>
   <child link="L_Pipe_1"/>
 </joint>
-<joint name="Rev61" type="continuous">
+<joint name="FR_1" type="continuous">
   <origin rpy="0 0 0" xyz="-0.054447 0.0 -0.054447"/>
   <parent link="FR_motor_block_1"/>
@@ -382,5 +380,5 @@
   <axis xyz="-0.0 -1.0 0.0"/>
 </joint>
-<joint name="Rev62" type="continuous">
+<joint name="FR_2" type="continuous">
   <origin rpy="0 0 0" xyz="0.0164 -0.075469 -0.051319"/>
   <parent link="FR_top_1"/>
