Commit message: New working URDF from @SpaceMaster85 exporter

File: ROS_Stack/src/zeta_urdf_description/urdf/materials.xacro (robot description, xacro)
@@ -1,6 +1,12 @@
 <?xml version="1.0" ?>
 <robot name="zeta_urdf" xmlns:xacro="http://www.ros.org/wiki/xacro" >
-<material name="silver">
+<material name="silver_default">
   <color rgba="0.700 0.700 0.700 1.000"/>
 </material>
+<material name="opaque252525">
+  <color rgba="0.09803921568627451 0.09803921568627451 0.09803921568627451 1.0"/>
+</material>
+<material name="opaque246246243">
+  <color rgba="0.9647058823529412 0.9647058823529412 0.9529411764705882 1.0"/>
+</material>
 </robot>

File: ROS_Stack/src/zeta_urdf_description/urdf/zeta_urdf.xacro (robot description, xacro)
@@ -6,17 +6,17 @@
 <link name="base_link">
   <inertial>
-    <origin rpy="0 0 0" xyz="0.5865154177311522 -0.47938007450948616 0.24225184206557204"/>
+    <origin xyz="0.5865154177311522 -0.47938007450948616 0.24225184206557204" rpy="0 0 0"/>
     <mass value="0.13102657430451126"/>
-    <inertia ixx="7e-05" ixy="0.0" ixz="-0.0" iyy="0.001452" iyz="-0.0" izz="0.001484"/>
-  </inertial>
-  <visual>
-    <origin rpy="0 0 0" xyz="0 0 0"/>
+    <inertia ixx="7e-05" iyy="0.001452" izz="0.001484" ixy="0.0" iyz="-0.0" ixz="-0.0"/>
+  </inertial>
+  <visual>
+    <origin xyz="0 0 0" rpy="0 0 0"/>
     <geometry>
       <mesh filename="package://zeta_urdf_description/meshes/base_link.stl" scale="0.001 0.001 0.001"/>
     </geometry>
-    <material name="silver"/>
-  </visual>
-  <collision>
-    <origin rpy="0 0 0" xyz="0 0 0"/>
+    <material name="opaque252525"/>
+  </visual>
+  <collision>
+    <origin xyz="0 0 0" rpy="0 0 0"/>
     <geometry>
       <mesh filename="package://zeta_urdf_description/meshes/base_link.stl" scale="0.001 0.001 0.001"/>
@@ -26,17 +26,17 @@
 <link name="FL_Foot_1">
   <inertial>
-    <origin rpy="0 0 0" xyz="-0.33499306627965986 -0.6826221079562163 -0.056449484510780606"/>
+    <origin xyz="0.05644893372034021 -0.015447107956216288 -0.056449484510780606" rpy="0 0 0"/>
     <mass value="0.050254366164942214"/>
-    <inertia ixx="4e-05" ixy="0.0" ixz="3.4e-05" iyy="7.1e-05" iyz="-0.0" izz="4e-05"/>
-  </inertial>
-  <visual>
-    <origin rpy="0 0 0" xyz="-1.058618 -0.302214 -0.136492"/>
+    <inertia ixx="4e-05" iyy="7.1e-05" izz="4e-05" ixy="0.0" iyz="-0.0" ixz="3.4e-05"/>
+  </inertial>
+  <visual>
+    <origin xyz="-0.667176 0.364961 -0.136492" rpy="0 0 0"/>
     <geometry>
       <mesh filename="package://zeta_urdf_description/meshes/FL_Foot_1.stl" scale="0.001 0.001 0.001"/>
     </geometry>
-    <material name="silver"/>
-  </visual>
-  <collision>
-    <origin rpy="0 0 0" xyz="-1.058618 -0.302214 -0.136492"/>
+    <material name="opaque252525"/>
+  </visual>
+  <collision>
+    <origin xyz="-0.667176 0.364961 -0.136492" rpy="0 0 0"/>
     <geometry>
       <mesh filename="package://zeta_urdf_description/meshes/FL_Foot_1.stl" scale="0.001 0.001 0.001"/>
@@ -46,17 +46,17 @@
 <link name="FL_Dual_Motor_Mount_1">
   <inertial>
-    <origin rpy="0 0 0" xyz="-0.37854432295995344 -0.7269301266658466 -0.017857804520426318"/>
+    <origin xyz="-0.01785632295995343 -1.2666584658926894e-07 -0.01785880452042632" rpy="0 0 0"/>
     <mass value="0.023417593270727483"/>
-    <inertia ixx="1.4e-05" ixy="0.0" ixz="-8e-06" iyy="2.5e-05" iyz="0.0" izz="1.4e-05"/>
-  </inertial>
-  <visual>
-    <origin rpy="0 0 0" xyz="-1.073118 -0.347469 -0.181746"/>
+    <inertia ixx="1.4e-05" iyy="2.5e-05" izz="1.4e-05" ixy="0.0" iyz="0.0" ixz="-8e-06"/>
+  </inertial>
+  <visual>
+    <origin xyz="-0.71243 0.379461 -0.181747" rpy="0 0 0"/>
     <geometry>
       <mesh filename="package://zeta_urdf_description/meshes/FL_Dual_Motor_Mount_1.stl" scale="0.001 0.001 0.001"/>
     </geometry>
-    <material name="silver"/>
-  </visual>
-  <collision>
-    <origin rpy="0 0 0" xyz="-1.073118 -0.347469 -0.181746"/>
+    <material name="opaque252525"/>
+  </visual>
+  <collision>
+    <origin xyz="-0.71243 0.379461 -0.181747" rpy="0 0 0"/>
     <geometry>
       <mesh filename="package://zeta_urdf_description/meshes/FL_Dual_Motor_Mount_1.stl" scale="0.001 0.001 0.001"/>
@@ -66,17 +66,17 @@
 <link name="FL_Top_Bracket_1">
   <inertial>
-    <origin rpy="0 0 0" xyz="-0.4121010303411867 -0.7331212860562331 -0.011363759328014672"/>
+    <origin xyz="0.015262969658813352 0.04757071394376694 -0.011363759328014672" rpy="0 0 0"/>
     <mass value="0.026371988478740775"/>
-    <inertia ixx="2.3e-05" ixy="-0.0" ixz="0.0" iyy="1.1e-05" iyz="4e-06" izz="1.8e-05"/>
-  </inertial>
-  <visual>
-    <origin rpy="0 0 0" xyz="-1.133337 -0.341012 -0.242258"/>
+    <inertia ixx="2.3e-05" iyy="1.1e-05" izz="1.8e-05" ixy="-0.0" iyz="4e-06" ixz="0.0"/>
+  </inertial>
+  <visual>
+    <origin xyz="-0.705973 0.43968 -0.242258" rpy="0 0 0"/>
     <geometry>
       <mesh filename="package://zeta_urdf_description/meshes/FL_Top_Bracket_1.stl" scale="0.001 0.001 0.001"/>
     </geometry>
-    <material name="silver"/>
-  </visual>
-  <collision>
-    <origin rpy="0 0 0" xyz="-1.133337 -0.341012 -0.242258"/>
+    <material name="opaque252525"/>
+  </visual>
+  <collision>
+    <origin xyz="-0.705973 0.43968 -0.242258" rpy="0 0 0"/>
     <geometry>
       <mesh filename="package://zeta_urdf_description/meshes/FL_Top_Bracket_1.stl" scale="0.001 0.001 0.001"/>
@@ -86,17 +86,17 @@
 <link name="FR_Top_Bracket_1">
   <inertial>
-    <origin rpy="0 0 0" xyz="-0.49150103034118864 -0.9076628629628037 -0.011363759328016143"/>
+    <origin xyz="0.015262969658811354 -0.04757086296280377 -0.011363759328016143" rpy="0 0 0"/>
     <mass value="0.02637198847874129"/>
-    <inertia ixx="2.3e-05" ixy="0.0" ixz="0.0" iyy="1.1e-05" iyz="-4e-06" izz="1.8e-05"/>
-  </inertial>
-  <visual>
-    <origin rpy="0 0 0" xyz="-1.212737 -0.341012 -0.242258"/>
+    <inertia ixx="2.3e-05" iyy="1.1e-05" izz="1.8e-05" ixy="0.0" iyz="-4e-06" ixz="0.0"/>
+  </inertial>
+  <visual>
+    <origin xyz="-0.705973 0.51908 -0.242258" rpy="0 0 0"/>
     <geometry>
       <mesh filename="package://zeta_urdf_description/meshes/FR_Top_Bracket_1.stl" scale="0.001 0.001 0.001"/>
     </geometry>
-    <material name="silver"/>
-  </visual>
-  <collision>
-    <origin rpy="0 0 0" xyz="-1.212737 -0.341012 -0.242258"/>
+    <material name="opaque252525"/>
+  </visual>
+  <collision>
+    <origin xyz="-0.705973 0.51908 -0.242258" rpy="0 0 0"/>
     <geometry>
       <mesh filename="package://zeta_urdf_description/meshes/FR_Top_Bracket_1.stl" scale="0.001 0.001 0.001"/>
@@ -106,17 +106,17 @@
 <link name="FR_3_Motor_1">
   <inertial>
-    <origin rpy="0 0 0" xyz="-0.48253131701923535 -0.8612109120079297 -4.0692889397009324e-07"/>
+    <origin xyz="0.00023268298076450922 0.00388108799207032 -4.0692889397009324e-07" rpy="0 0 0"/>
     <mass value="0.26893718656206705"/>
-    <inertia ixx="5.9e-05" ixy="0.0" ixz="-0.0" iyy="3.6e-05" iyz="-0.0" izz="6.8e-05"/>
-  </inertial>
-  <visual>
-    <origin rpy="0 0 0" xyz="-1.203237 -0.355512 -0.242258"/>
+    <inertia ixx="5.9e-05" iyy="3.6e-05" izz="6.8e-05" ixy="0.0" iyz="-0.0" ixz="-0.0"/>
+  </inertial>
+  <visual>
+    <origin xyz="-0.720473 0.50958 -0.242258" rpy="0 0 0"/>
     <geometry>
       <mesh filename="package://zeta_urdf_description/meshes/FR_3_Motor_1.stl" scale="0.001 0.001 0.001"/>
     </geometry>
-    <material name="silver"/>
-  </visual>
-  <collision>
-    <origin rpy="0 0 0" xyz="-1.203237 -0.355512 -0.242258"/>
+    <material name="opaque252525"/>
+  </visual>
+  <collision>
+    <origin xyz="-0.720473 0.50958 -0.242258" rpy="0 0 0"/>
     <geometry>
       <mesh filename="package://zeta_urdf_description/meshes/FR_3_Motor_1.stl" scale="0.001 0.001 0.001"/>
@@ -126,17 +126,17 @@
 <link name="Pipe_R_1">
   <inertial>
-    <origin rpy="0 0 0" xyz="0.1149248413410463 -0.0001969694373666897 1.862640597316556e-10"/>
+    <origin xyz="0.1149248413410463 -0.0001969694373666897 1.862640597316556e-10" rpy="0 0 0"/>
     <mass value="0.060722328485887364"/>
-    <inertia ixx="5e-06" ixy="0.0" ixz="0.0" iyy="0.00027" iyz="0.0" izz="0.00027"/>
-  </inertial>
-  <visual>
-    <origin rpy="0 0 0" xyz="-0.469873 0.499765 -0.242258"/>
+    <inertia ixx="5e-06" iyy="0.00027" izz="0.00027" ixy="0.0" iyz="0.0" ixz="0.0"/>
+  </inertial>
+  <visual>
+    <origin xyz="-0.469873 0.499765 -0.242258" rpy="0 0 0"/>
     <geometry>
       <mesh filename="package://zeta_urdf_description/meshes/Pipe_R_1.stl" scale="0.001 0.001 0.001"/>
     </geometry>
-    <material name="silver"/>
-  </visual>
-  <collision>
-    <origin rpy="0 0 0" xyz="-0.469873 0.499765 -0.242258"/>
+    <material name="opaque246246243"/>
+  </visual>
+  <collision>
+    <origin xyz="-0.469873 0.499765 -0.242258" rpy="0 0 0"/>
     <geometry>
       <mesh filename="package://zeta_urdf_description/meshes/Pipe_R_1.stl" scale="0.001 0.001 0.001"/>
@@ -146,17 +146,17 @@
 <link name="Pipe_L_1">
   <inertial>
-    <origin rpy="0 0 0" xyz="0.11492484134104641 0.0001968204183980804 1.8626425402068492e-10"/>
+    <origin xyz="0.11492484134104641 0.0001968204183980804 1.8626425402068492e-10" rpy="0 0 0"/>
     <mass value="0.06072232848588741"/>
-    <inertia ixx="5e-06" ixy="0.0" ixz="-0.0" iyy="0.00027" iyz="0.0" izz="0.00027"/>
-  </inertial>
-  <visual>
-    <origin rpy="0 0 0" xyz="-0.469873 0.458995 -0.242258"/>
+    <inertia ixx="5e-06" iyy="0.00027" izz="0.00027" ixy="0.0" iyz="0.0" ixz="-0.0"/>
+  </inertial>
+  <visual>
+    <origin xyz="-0.469873 0.458995 -0.242258" rpy="0 0 0"/>
     <geometry>
       <mesh filename="package://zeta_urdf_description/meshes/Pipe_L_1.stl" scale="0.001 0.001 0.001"/>
     </geometry>
-    <material name="silver"/>
-  </visual>
-  <collision>
-    <origin rpy="0 0 0" xyz="-0.469873 0.458995 -0.242258"/>
+    <material name="opaque246246243"/>
+  </visual>
+  <collision>
+    <origin xyz="-0.469873 0.458995 -0.242258" rpy="0 0 0"/>
     <geometry>
       <mesh filename="package://zeta_urdf_description/meshes/Pipe_L_1.stl" scale="0.001 0.001 0.001"/>
@@ -166,17 +166,17 @@
 <link name="BR_3_Motor_1">
   <inertial>
-    <origin rpy="0 0 0" xyz="-0.7535313170189281 -0.5902109120079267 -4.0692889261007004e-07"/>
+    <origin xyz="0.00023268298107181895 0.0038810879920733177 -4.0692889261007004e-07" rpy="0 0 0"/>
     <mass value="0.26893718656206766"/>
-    <inertia ixx="5.9e-05" ixy="0.0" ixz="-0.0" iyy="3.6e-05" iyz="-0.0" izz="6.8e-05"/>
-  </inertial>
-  <visual>
-    <origin rpy="0 0 0" xyz="-1.203237 -0.084512 -0.242258"/>
+    <inertia ixx="5.9e-05" iyy="3.6e-05" izz="6.8e-05" ixy="0.0" iyz="-0.0" ixz="-0.0"/>
+  </inertial>
+  <visual>
+    <origin xyz="-0.449473 0.50958 -0.242258" rpy="0 0 0"/>
     <geometry>
       <mesh filename="package://zeta_urdf_description/meshes/BR_3_Motor_1.stl" scale="0.001 0.001 0.001"/>
     </geometry>
-    <material name="silver"/>
-  </visual>
-  <collision>
-    <origin rpy="0 0 0" xyz="-1.203237 -0.084512 -0.242258"/>
+    <material name="opaque252525"/>
+  </visual>
+  <collision>
+    <origin xyz="-0.449473 0.50958 -0.242258" rpy="0 0 0"/>
     <geometry>
       <mesh filename="package://zeta_urdf_description/meshes/BR_3_Motor_1.stl" scale="0.001 0.001 0.001"/>
@@ -186,17 +186,17 @@
 <link name="BL_3_Motor_1">
   <inertial>
-    <origin rpy="0 0 0" xyz="-0.6931313170189266 -0.5375732370107782 -4.0692889305415925e-07"/>
+    <origin xyz="0.00023268298107342877 -0.0038812370107781935 -4.0692889305415925e-07" rpy="0 0 0"/>
     <mass value="0.26893718656206744"/>
-    <inertia ixx="5.9e-05" ixy="-0.0" ixz="-0.0" iyy="3.6e-05" iyz="0.0" izz="6.8e-05"/>
-  </inertial>
-  <visual>
-    <origin rpy="0 0 0" xyz="-1.142837 -0.084512 -0.242258"/>
+    <inertia ixx="5.9e-05" iyy="3.6e-05" izz="6.8e-05" ixy="-0.0" iyz="0.0" ixz="-0.0"/>
+  </inertial>
+  <visual>
+    <origin xyz="-0.449473 0.44918 -0.242258" rpy="0 0 0"/>
     <geometry>
       <mesh filename="package://zeta_urdf_description/meshes/BL_3_Motor_1.stl" scale="0.001 0.001 0.001"/>
     </geometry>
-    <material name="silver"/>
-  </visual>
-  <collision>
-    <origin rpy="0 0 0" xyz="-1.142837 -0.084512 -0.242258"/>
+    <material name="opaque252525"/>
+  </visual>
+  <collision>
+    <origin xyz="-0.449473 0.44918 -0.242258" rpy="0 0 0"/>
     <geometry>
       <mesh filename="package://zeta_urdf_description/meshes/BL_3_Motor_1.stl" scale="0.001 0.001 0.001"/>
@@ -206,17 +206,17 @@
 <link name="BR_Top_Bracket_1">
   <inertial>
-    <origin rpy="0 0 0" xyz="-0.7625010303412662 -0.6366628629627984 -0.011363759328014672"/>
+    <origin xyz="0.015262969658733805 -0.047570862962798444 -0.011363759328014672" rpy="0 0 0"/>
     <mass value="0.026371988478740113"/>
-    <inertia ixx="2.3e-05" ixy="0.0" ixz="0.0" iyy="1.1e-05" iyz="-4e-06" izz="1.8e-05"/>
-  </inertial>
-  <visual>
-    <origin rpy="0 0 0" xyz="-1.212737 -0.070012 -0.242258"/>
+    <inertia ixx="2.3e-05" iyy="1.1e-05" izz="1.8e-05" ixy="0.0" iyz="-4e-06" ixz="0.0"/>
+  </inertial>
+  <visual>
+    <origin xyz="-0.434973 0.51908 -0.242258" rpy="0 0 0"/>
     <geometry>
       <mesh filename="package://zeta_urdf_description/meshes/BR_Top_Bracket_1.stl" scale="0.001 0.001 0.001"/>
     </geometry>
-    <material name="silver"/>
-  </visual>
-  <collision>
-    <origin rpy="0 0 0" xyz="-1.212737 -0.070012 -0.242258"/>
+    <material name="opaque252525"/>
+  </visual>
+  <collision>
+    <origin xyz="-0.434973 0.51908 -0.242258" rpy="0 0 0"/>
     <geometry>
       <mesh filename="package://zeta_urdf_description/meshes/BR_Top_Bracket_1.stl" scale="0.001 0.001 0.001"/>
@@ -226,17 +226,17 @@
 <link name="BL_Dual_Motor_Mount_1">
   <inertial>
-    <origin rpy="0 0 0" xyz="-0.6497187698347413 -0.455930126665844 -0.018030558804326358"/>
+    <origin xyz="-0.018030769834741278 -1.2666584398024483e-07 -0.01803155880432636" rpy="0 0 0"/>
     <mass value="0.02330043804692393"/>
-    <inertia ixx="1.4e-05" ixy="0.0" ixz="-8e-06" iyy="2.5e-05" iyz="0.0" izz="1.4e-05"/>
-  </inertial>
-  <visual>
-    <origin rpy="0 0 0" xyz="-1.073118 -0.076469 -0.181746"/>
+    <inertia ixx="1.4e-05" iyy="2.5e-05" izz="1.4e-05" ixy="0.0" iyz="0.0" ixz="-8e-06"/>
+  </inertial>
+  <visual>
+    <origin xyz="-0.44143 0.379461 -0.181747" rpy="0 0 0"/>
     <geometry>
       <mesh filename="package://zeta_urdf_description/meshes/BL_Dual_Motor_Mount_1.stl" scale="0.001 0.001 0.001"/>
     </geometry>
-    <material name="silver"/>
-  </visual>
-  <collision>
-    <origin rpy="0 0 0" xyz="-1.073118 -0.076469 -0.181746"/>
+    <material name="opaque252525"/>
+  </visual>
+  <collision>
+    <origin xyz="-0.44143 0.379461 -0.181747" rpy="0 0 0"/>
     <geometry>
       <mesh filename="package://zeta_urdf_description/meshes/BL_Dual_Motor_Mount_1.stl" scale="0.001 0.001 0.001"/>
@@ -246,17 +246,17 @@
 <link name="BL_Top_Bracket_1">
   <inertial>
-    <origin rpy="0 0 0" xyz="-0.6831010303412655 -0.4621212860562303 -0.01136375932801384"/>
+    <origin xyz="0.015262969658734526 0.047570713943769716 -0.01136375932801384" rpy="0 0 0"/>
     <mass value="0.02637198847874093"/>
-    <inertia ixx="2.3e-05" ixy="-0.0" ixz="0.0" iyy="1.1e-05" iyz="4e-06" izz="1.8e-05"/>
-  </inertial>
-  <visual>
-    <origin rpy="0 0 0" xyz="-1.133337 -0.070012 -0.242258"/>
+    <inertia ixx="2.3e-05" iyy="1.1e-05" izz="1.8e-05" ixy="-0.0" iyz="4e-06" ixz="0.0"/>
+  </inertial>
+  <visual>
+    <origin xyz="-0.434973 0.43968 -0.242258" rpy="0 0 0"/>
     <geometry>
       <mesh filename="package://zeta_urdf_description/meshes/BL_Top_Bracket_1.stl" scale="0.001 0.001 0.001"/>
     </geometry>
-    <material name="silver"/>
-  </visual>
-  <collision>
-    <origin rpy="0 0 0" xyz="-1.133337 -0.070012 -0.242258"/>
+    <material name="opaque252525"/>
+  </visual>
+  <collision>
+    <origin xyz="-0.434973 0.43968 -0.242258" rpy="0 0 0"/>
     <geometry>
       <mesh filename="package://zeta_urdf_description/meshes/BL_Top_Bracket_1.stl" scale="0.001 0.001 0.001"/>
@@ -266,17 +266,17 @@
 <link name="FL_2_Motor_1">
   <inertial>
-    <origin rpy="0 0 0" xyz="-0.34570678163021107 -0.7363559683056364 -0.009462146346697065"/>
+    <origin xyz="-0.009461781630211052 -0.015482968305636502 -0.009462146346697065" rpy="0 0 0"/>
     <mass value="0.26893718656110227"/>
-    <inertia ixx="5.2e-05" ixy="0.0" ixz="-1.6e-05" iyy="5.9e-05" iyz="0.0" izz="5.2e-05"/>
-  </inertial>
-  <visual>
-    <origin rpy="0 0 0" xyz="-1.057868 -0.356662 -0.190939"/>
+    <inertia ixx="5.2e-05" iyy="5.9e-05" izz="5.2e-05" ixy="0.0" iyz="0.0" ixz="-1.6e-05"/>
+  </inertial>
+  <visual>
+    <origin xyz="-0.721623 0.364211 -0.190939" rpy="0 0 0"/>
     <geometry>
       <mesh filename="package://zeta_urdf_description/meshes/FL_2_Motor_1.stl" scale="0.001 0.001 0.001"/>
     </geometry>
-    <material name="silver"/>
-  </visual>
-  <collision>
-    <origin rpy="0 0 0" xyz="-1.057868 -0.356662 -0.190939"/>
+    <material name="opaque252525"/>
+  </visual>
+  <collision>
+    <origin xyz="-0.721623 0.364211 -0.190939" rpy="0 0 0"/>
     <geometry>
       <mesh filename="package://zeta_urdf_description/meshes/FL_2_Motor_1.stl" scale="0.001 0.001 0.001"/>
@@ -286,17 +286,17 @@
 <link name="FL_1_Motor_1">
   <inertial>
-    <origin rpy="0 0 0" xyz="-0.3964807580392644 -0.6886259683056364 0.00274502873903551"/>
+    <origin xyz="0.0027442419607356383 -0.00023296830563640514 0.00274502873903551" rpy="0 0 0"/>
     <mass value="0.26893718656110227"/>
-    <inertia ixx="5.2e-05" ixy="-0.0" ixz="-1.6e-05" iyy="5.9e-05" iyz="-0.0" izz="5.2e-05"/>
-  </inertial>
-  <visual>
-    <origin rpy="0 0 0" xyz="-1.073118 -0.308932 -0.143209"/>
+    <inertia ixx="5.2e-05" iyy="5.9e-05" izz="5.2e-05" ixy="-0.0" iyz="-0.0" ixz="-1.6e-05"/>
+  </inertial>
+  <visual>
+    <origin xyz="-0.673893 0.379461 -0.143209" rpy="0 0 0"/>
     <geometry>
       <mesh filename="package://zeta_urdf_description/meshes/FL_1_Motor_1.stl" scale="0.001 0.001 0.001"/>
     </geometry>
-    <material name="silver"/>
-  </visual>
-  <collision>
-    <origin rpy="0 0 0" xyz="-1.073118 -0.308932 -0.143209"/>
+    <material name="opaque252525"/>
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