Commit message: Update tuned URDF to have new I clamp in the URDF folder

File: URDF/Tuned_URDF/zeta_urdf_description/urdf/zeta_urdf.xacro (robot description, xacro)
@@ -1,25 +1,16 @@
 <?xml version="1.0" ?>
 <robot name="zeta_urdf" xmlns:xacro="http://www.ros.org/wiki/xacro">
-<material name="silver_default">
-  <color rgba="0.700 0.700 0.700 1.000"/>
-</material>
-<material name="opaque252525">
-  <color rgba="0.09803921568627451 0.09803921568627451 0.09803921568627451 1.0"/>
-</material>
-<material name="opaque246246243">
-  <color rgba="0.9647058823529412 0.9647058823529412 0.9529411764705882 1.0"/>
-</material>
+<xacro:include filename="$(find zeta_urdf_description)/urdf/materials.xacro" />
 <xacro:include filename="$(find zeta_urdf_description)/urdf/zeta_urdf.trans" />
 <xacro:include filename="$(find zeta_urdf_description)/urdf/zeta_urdf.gazebo" />
+<xacro:property name="damping_value" value="50" />
+<xacro:property name="friction_value" value="0.1" />
 <link name="dummy">
    </link>
 <link name="base_link">
   <inertial>
-    <origin xyz="0.5865154177311522 -0.47938007450948616 0.24225184206557204" rpy="0 0 0"/>
+    <origin xyz="-0.006887732149199177 0.005649968016768892 0.20576830530971255" rpy="0 0 0"/>
     <mass value="0.13102657430451126"/>
-    <inertia ixx="0.0001" ixy="0.000"  ixz="0.000"
-         iyy="0.0001" iyz="0.000"
-         izz="0.0001"
-/>
+    <inertia ixx="7e-05" iyy="0.001452" izz="0.001484" ixy="0.0" iyz="-0.0" ixz="-0.0"/>
   </inertial>
   <visual>
@@ -43,13 +34,10 @@
 <link name="FL_Foot_1">
   <inertial>
-    <origin xyz="0.05644893372034021 -0.015447107956216288 -0.056449484510780606" rpy="0 0 0"/>
-    <mass value="0.050254366164942214"/>
-    <inertia ixx="0.0001" ixy="0.000"  ixz="0.000"
-         iyy="0.0001" iyz="0.000"
-         izz="0.0001"
-/>
-  </inertial>
-  <visual>
-    <origin xyz="-0.667176 0.364961 -0.136492" rpy="0 0 0"/>
+    <origin xyz="0.05628492645882191 -0.015254964193953696 -0.06460044311982074" rpy="0 0 0"/>
+    <mass value="0.10306892931910153"/>
+    <inertia ixx="0.000157" iyy="0.000228" izz="8.7e-05" ixy="0.0" iyz="-0.0" ixz="9.8e-05"/>
+  </inertial>
+  <visual>
+    <origin xyz="-0.073772 -0.120069 -0.100008" rpy="0 0 0"/>
     <geometry>
       <mesh filename="package://zeta_urdf_description/meshes/FL_Foot_1.stl" scale="0.001 0.001 0.001"/>
@@ -58,5 +46,5 @@
   </visual>
   <collision>
-    <origin xyz="-0.667176 0.364961 -0.136492" rpy="0 0 0"/>
+    <origin xyz="-0.073772 -0.120069 -0.100008" rpy="0 0 0"/>
     <geometry>
       <mesh filename="package://zeta_urdf_description/meshes/FL_Foot_1.stl" scale="0.001 0.001 0.001"/>
@@ -66,13 +54,10 @@
 <link name="FL_Dual_Motor_Mount_1">
   <inertial>
-    <origin xyz="-0.01785632295995343 -1.2666584658926894e-07 -0.01785880452042632" rpy="0 0 0"/>
+    <origin xyz="-0.0178564728403042 -8.413959165509688e-08 -0.01785834127628591" rpy="0 0 0"/>
     <mass value="0.023417593270727483"/>
-    <inertia ixx="0.0001" ixy="0.000"  ixz="0.000"
-         iyy="0.0001" iyz="0.000"
-         izz="0.0001"
-/>
-  </inertial>
-  <visual>
-    <origin xyz="-0.71243 0.379461 -0.181747" rpy="0 0 0"/>
+    <inertia ixx="1.4e-05" iyy="2.5e-05" izz="1.4e-05" ixy="0.0" iyz="-0.0" ixz="-8e-06"/>
+  </inertial>
+  <visual>
+    <origin xyz="-0.119027 -0.105569 -0.145263" rpy="0 0 0"/>
     <geometry>
       <mesh filename="package://zeta_urdf_description/meshes/FL_Dual_Motor_Mount_1.stl" scale="0.001 0.001 0.001"/>
@@ -81,5 +66,5 @@
   </visual>
   <collision>
-    <origin xyz="-0.71243 0.379461 -0.181747" rpy="0 0 0"/>
+    <origin xyz="-0.119027 -0.105569 -0.145263" rpy="0 0 0"/>
     <geometry>
       <mesh filename="package://zeta_urdf_description/meshes/FL_Dual_Motor_Mount_1.stl" scale="0.001 0.001 0.001"/>
@@ -89,13 +74,10 @@
 <link name="FL_Top_Bracket_1">
   <inertial>
-    <origin xyz="0.015262969658813352 0.04757071394376694 -0.011363759328014672" rpy="0 0 0"/>
+    <origin xyz="0.015262819778462638 0.04757075647002189 -0.011363296083874236" rpy="0 0 0"/>
     <mass value="0.026371988478740775"/>
-    <inertia ixx="0.0001" ixy="0.000"  ixz="0.000"
-         iyy="0.0001" iyz="0.000"
-         izz="0.0001"
-/>
-  </inertial>
-  <visual>
-    <origin xyz="-0.705973 0.43968 -0.242258" rpy="0 0 0"/>
+    <inertia ixx="2.3e-05" iyy="1.1e-05" izz="1.8e-05" ixy="-0.0" iyz="4e-06" ixz="0.0"/>
+  </inertial>
+  <visual>
+    <origin xyz="-0.11257 -0.04535 -0.205774" rpy="0 0 0"/>
     <geometry>
       <mesh filename="package://zeta_urdf_description/meshes/FL_Top_Bracket_1.stl" scale="0.001 0.001 0.001"/>
@@ -104,5 +86,5 @@
   </visual>
   <collision>
-    <origin xyz="-0.705973 0.43968 -0.242258" rpy="0 0 0"/>
+    <origin xyz="-0.11257 -0.04535 -0.205774" rpy="0 0 0"/>
     <geometry>
       <mesh filename="package://zeta_urdf_description/meshes/FL_Top_Bracket_1.stl" scale="0.001 0.001 0.001"/>
@@ -112,13 +94,10 @@
 <link name="FR_Top_Bracket_1">
   <inertial>
-    <origin xyz="0.015262969658811354 -0.04757086296280377 -0.011363759328016143" rpy="0 0 0"/>
+    <origin xyz="0.015262819778460085 -0.04757082043654881 -0.011363296083875513" rpy="0 0 0"/>
     <mass value="0.02637198847874129"/>
-    <inertia ixx="0.0001" ixy="0.000"  ixz="0.000"
-         iyy="0.0001" iyz="0.000"
-         izz="0.0001"
-/>
-  </inertial>
-  <visual>
-    <origin xyz="-0.705973 0.51908 -0.242258" rpy="0 0 0"/>
+    <inertia ixx="2.3e-05" iyy="1.1e-05" izz="1.8e-05" ixy="0.0" iyz="-4e-06" ixz="0.0"/>
+  </inertial>
+  <visual>
+    <origin xyz="-0.11257 0.03405 -0.205774" rpy="0 0 0"/>
     <geometry>
       <mesh filename="package://zeta_urdf_description/meshes/FR_Top_Bracket_1.stl" scale="0.001 0.001 0.001"/>
@@ -127,5 +106,5 @@
   </visual>
   <collision>
-    <origin xyz="-0.705973 0.51908 -0.242258" rpy="0 0 0"/>
+    <origin xyz="-0.11257 0.03405 -0.205774" rpy="0 0 0"/>
     <geometry>
       <mesh filename="package://zeta_urdf_description/meshes/FR_Top_Bracket_1.stl" scale="0.001 0.001 0.001"/>
@@ -135,13 +114,10 @@
 <link name="FR_3_Motor_1">
   <inertial>
-    <origin xyz="0.00023268298076450922 0.00388108799207032 -4.069288939978488e-07" rpy="0 0 0"/>
+    <origin xyz="0.0002325331004134623 0.0038811305183252993 5.631524657712106e-08" rpy="0 0 0"/>
     <mass value="0.09250068837166636"/>
-    <inertia ixx="0.0001" ixy="0.000"  ixz="0.000"
-         iyy="0.0001" iyz="0.000"
-         izz="0.0001"
-/>
-  </inertial>
-  <visual>
-    <origin xyz="-0.720473 0.50958 -0.242258" rpy="0 0 0"/>
+    <inertia ixx="2e-05" iyy="1.2e-05" izz="2.3e-05" ixy="0.0" iyz="-0.0" ixz="-0.0"/>
+  </inertial>
+  <visual>
+    <origin xyz="-0.12707 0.02455 -0.205774" rpy="0 0 0"/>
     <geometry>
       <mesh filename="package://zeta_urdf_description/meshes/FR_3_Motor_1.stl" scale="0.001 0.001 0.001"/>
@@ -150,5 +126,5 @@
   </visual>
   <collision>
-    <origin xyz="-0.720473 0.50958 -0.242258" rpy="0 0 0"/>
+    <origin xyz="-0.12707 0.02455 -0.205774" rpy="0 0 0"/>
     <geometry>
       <mesh filename="package://zeta_urdf_description/meshes/FR_3_Motor_1.stl" scale="0.001 0.001 0.001"/>
@@ -158,13 +134,10 @@
 <link name="Pipe_R_1">
   <inertial>
-    <origin xyz="0.1149248413410463 -0.0001969694373666897 1.862640597316556e-10" rpy="0 0 0"/>
+    <origin xyz="0.11492469146069478 -0.00019692691111165318 4.6343040452367923e-07" rpy="0 0 0"/>
     <mass value="0.060722328485887364"/>
-    <inertia ixx="0.0001" ixy="0.000"  ixz="0.000"
-         iyy="0.0001" iyz="0.000"
-         izz="0.0001"
-/>
-  </inertial>
-  <visual>
-    <origin xyz="-0.469873 0.499765 -0.242258" rpy="0 0 0"/>
+    <inertia ixx="5e-06" iyy="0.00027" izz="0.00027" ixy="0.0" iyz="-0.0" ixz="-0.0"/>
+  </inertial>
+  <visual>
+    <origin xyz="0.12353 0.014735 -0.205774" rpy="0 0 0"/>
     <geometry>
       <mesh filename="package://zeta_urdf_description/meshes/Pipe_R_1.stl" scale="0.001 0.001 0.001"/>
@@ -173,5 +146,5 @@
   </visual>
   <collision>
-    <origin xyz="-0.469873 0.499765 -0.242258" rpy="0 0 0"/>
+    <origin xyz="0.12353 0.014735 -0.205774" rpy="0 0 0"/>
     <geometry>
       <mesh filename="package://zeta_urdf_description/meshes/Pipe_R_1.stl" scale="0.001 0.001 0.001"/>
@@ -181,13 +154,10 @@
 <link name="Pipe_L_1">
   <inertial>
-    <origin xyz="0.11492484134104641 0.0001968204183980804 1.8626425402068492e-10" rpy="0 0 0"/>
+    <origin xyz="0.11492469146069506 0.00019686294465318457 4.634304046902127e-07" rpy="0 0 0"/>
     <mass value="0.06072232848588741"/>
-    <inertia ixx="0.0001" ixy="0.000"  ixz="0.000"
-         iyy="0.0001" iyz="0.000"
-         izz="0.0001"
-/>
-  </inertial>
-  <visual>
-    <origin xyz="-0.469873 0.458995 -0.242258" rpy="0 0 0"/>
+    <inertia ixx="5e-06" iyy="0.00027" izz="0.00027" ixy="0.0" iyz="-0.0" ixz="-0.0"/>
+  </inertial>
+  <visual>
+    <origin xyz="0.12353 -0.026035 -0.205774" rpy="0 0 0"/>
     <geometry>
       <mesh filename="package://zeta_urdf_description/meshes/Pipe_L_1.stl" scale="0.001 0.001 0.001"/>
@@ -196,5 +166,5 @@
   </visual>
   <collision>
-    <origin xyz="-0.469873 0.458995 -0.242258" rpy="0 0 0"/>
+    <origin xyz="0.12353 -0.026035 -0.205774" rpy="0 0 0"/>
     <geometry>
       <mesh filename="package://zeta_urdf_description/meshes/Pipe_L_1.stl" scale="0.001 0.001 0.001"/>
@@ -204,13 +174,10 @@
 <link name="BR_3_Motor_1">
   <inertial>
-    <origin xyz="0.00023268298107181895 0.0038810879920733177 -4.0692889261007004e-07" rpy="0 0 0"/>
+    <origin xyz="0.0002325331007198006 0.0038811305183284427 5.6315247798366386e-08" rpy="0 0 0"/>
     <mass value="0.09250068837166658"/>
-    <inertia ixx="0.0001" ixy="0.000"  ixz="0.000"
-         iyy="0.0001" iyz="0.000"
-         izz="0.0001"
-/>
-  </inertial>
-  <visual>
-    <origin xyz="-0.449473 0.50958 -0.242258" rpy="0 0 0"/>
+    <inertia ixx="2e-05" iyy="1.2e-05" izz="2.3e-05" ixy="0.0" iyz="-0.0" ixz="-0.0"/>
+  </inertial>
+  <visual>
+    <origin xyz="0.14393 0.02455 -0.205774" rpy="0 0 0"/>
     <geometry>
       <mesh filename="package://zeta_urdf_description/meshes/BR_3_Motor_1.stl" scale="0.001 0.001 0.001"/>
@@ -219,5 +186,5 @@
   </visual>
   <collision>
-    <origin xyz="-0.449473 0.50958 -0.242258" rpy="0 0 0"/>
+    <origin xyz="0.14393 0.02455 -0.205774" rpy="0 0 0"/>
     <geometry>
       <mesh filename="package://zeta_urdf_description/meshes/BR_3_Motor_1.stl" scale="0.001 0.001 0.001"/>
@@ -227,13 +194,10 @@
 <link name="BL_3_Motor_1">
   <inertial>
-    <origin xyz="0.00023268298107342877 -0.0038812370107781935 -4.0692889305415925e-07" rpy="0 0 0"/>
+    <origin xyz="0.00023253310072163247 -0.003881194484523093 5.63152473265216e-08" rpy="0 0 0"/>
     <mass value="0.0925006883716665"/>
-    <inertia ixx="0.0001" ixy="0.000"  ixz="0.000"
-         iyy="0.0001" iyz="0.000"
-         izz="0.0001"
-/>
-  </inertial>
-  <visual>
-    <origin xyz="-0.449473 0.44918 -0.242258" rpy="0 0 0"/>
+    <inertia ixx="2e-05" iyy="1.2e-05" izz="2.3e-05" ixy="-0.0" iyz="0.0" ixz="-0.0"/>
+  </inertial>
+  <visual>
+    <origin xyz="0.14393 -0.03585 -0.205774" rpy="0 0 0"/>
     <geometry>
       <mesh filename="package://zeta_urdf_description/meshes/BL_3_Motor_1.stl" scale="0.001 0.001 0.001"/>
@@ -242,5 +206,5 @@
   </visual>
   <collision>
-    <origin xyz="-0.449473 0.44918 -0.242258" rpy="0 0 0"/>
+    <origin xyz="0.14393 -0.03585 -0.205774" rpy="0 0 0"/>
     <geometry>
       <mesh filename="package://zeta_urdf_description/meshes/BL_3_Motor_1.stl" scale="0.001 0.001 0.001"/>
@@ -250,13 +214,10 @@
 <link name="BR_Top_Bracket_1">
   <inertial>
-    <origin xyz="0.015262969658733805 -0.047570862962798444 -0.011363759328014672" rpy="0 0 0"/>
+    <origin xyz="0.015262819778381648 -0.04757082043654326 -0.01136329608387418" rpy="0 0 0"/>
     <mass value="0.026371988478740113"/>
-    <inertia ixx="0.0001" ixy="0.000"  ixz="0.000"
-         iyy="0.0001" iyz="0.000"
-         izz="0.0001"
-/>
-  </inertial>
-  <visual>
-    <origin xyz="-0.434973 0.51908 -0.242258" rpy="0 0 0"/>
+    <inertia ixx="2.3e-05" iyy="1.1e-05" izz="1.8e-05" ixy="0.0" iyz="-4e-06" ixz="0.0"/>
+  </inertial>
+  <visual>
+    <origin xyz="0.15843 0.03405 -0.205774" rpy="0 0 0"/>
     <geometry>
       <mesh filename="package://zeta_urdf_description/meshes/BR_Top_Bracket_1.stl" scale="0.001 0.001 0.001"/>
@@ -265,5 +226,5 @@
   </visual>
   <collision>
-    <origin xyz="-0.434973 0.51908 -0.242258" rpy="0 0 0"/>
+    <origin xyz="0.15843 0.03405 -0.205774" rpy="0 0 0"/>
     <geometry>
       <mesh filename="package://zeta_urdf_description/meshes/BR_Top_Bracket_1.stl" scale="0.001 0.001 0.001"/>
@@ -273,13 +234,10 @@
 <link name="BL_Dual_Motor_Mount_1">
   <inertial>
-    <origin xyz="-0.018030769834741278 -1.2666584398024483e-07 -0.01803155880432636" rpy="0 0 0"/>
+    <origin xyz="-0.018030919715092797 -8.413958881015038e-08 -0.018031095560186033" rpy="0 0 0"/>
     <mass value="0.02330043804692393"/>
-    <inertia ixx="0.0001" ixy="0.000"  ixz="0.000"
-         iyy="0.0001" iyz="0.000"
-         izz="0.0001"
-/>
-  </inertial>
-  <visual>
-    <origin xyz="-0.44143 0.379461 -0.181747" rpy="0 0 0"/>
+    <inertia ixx="1.4e-05" iyy="2.5e-05" izz="1.4e-05" ixy="0.0" iyz="-0.0" ixz="-8e-06"/>
+  </inertial>
+  <visual>
+    <origin xyz="0.151973 -0.105569 -0.145263" rpy="0 0 0"/>
     <geometry>
       <mesh filename="package://zeta_urdf_description/meshes/BL_Dual_Motor_Mount_1.stl" scale="0.001 0.001 0.001"/>
@@ -288,5 +246,5 @@
   </visual>
   <collision>
-    <origin xyz="-0.44143 0.379461 -0.181747" rpy="0 0 0"/>
+    <origin xyz="0.151973 -0.105569 -0.145263" rpy="0 0 0"/>
     <geometry>
       <mesh filename="package://zeta_urdf_description/meshes/BL_Dual_Motor_Mount_1.stl" scale="0.001 0.001 0.001"/>
@@ -296,13 +254,10 @@
 <link name="BL_Top_Bracket_1">
   <inertial>
-    <origin xyz="0.015262969658734526 0.047570713943769716 -0.01136375932801384" rpy="0 0 0"/>
+    <origin xyz="0.015262819778382924 0.04757075647002487 -0.011363296083873542" rpy="0 0 0"/>
     <mass value="0.02637198847874093"/>
-    <inertia ixx="0.0001" ixy="0.000"  ixz="0.000"
-         iyy="0.0001" iyz="0.000"
-         izz="0.0001"
-/>
-  </inertial>
-  <visual>
-    <origin xyz="-0.434973 0.43968 -0.242258" rpy="0 0 0"/>
+    <inertia ixx="2.3e-05" iyy="1.1e-05" izz="1.8e-05" ixy="-0.0" iyz="4e-06" ixz="0.0"/>
+  </inertial>
+  <visual>
+    <origin xyz="0.15843 -0.04535 -0.205774" rpy="0 0 0"/>
     <geometry>
       <mesh filename="package://zeta_urdf_description/meshes/BL_Top_Bracket_1.stl" scale="0.001 0.001 0.001"/>
@@ -311,5 +266,5 @@
   </visual>
   <collision>
-    <origin xyz="-0.434973 0.43968 -0.242258" rpy="0 0 0"/>
+    <origin xyz="0.15843 -0.04535 -0.205774" rpy="0 0 0"/>
     <geometry>
       <mesh filename="package://zeta_urdf_description/meshes/BL_Top_Bracket_1.stl" scale="0.001 0.001 0.001"/>
@@ -319,13 +274,10 @@
 <link name="FL_2_Motor_1">
   <inertial>
-    <origin xyz="-0.009461781630211052 -0.015482968305636502 -0.009462146346697065" rpy="0 0 0"/>
+    <origin xyz="-0.009461931510561628 -0.015482925779381568 -0.00946268310255663" rpy="0 0 0"/>
     <mass value="0.09250068837133453"/>
-    <inertia ixx="0.0001" ixy="0.000"  ixz="0.000"
-         iyy="0.0001" iyz="0.000"
-         izz="0.0001"
-/>
-  </inertial>
-  <visual>
-    <origin xyz="-0.721623 0.364211 -0.190939" rpy="0 0 0"/>
+    <inertia ixx="1.8e-05" iyy="2e-05" izz="1.8e-05" ixy="0.0" iyz="0.0" ixz="-5e-06"/>
+  </inertial>
+  <visual>
+    <origin xyz="-0.12822 -0.120819 -0.154456" rpy="0 0 0"/>
     <geometry>
       <mesh filename="package://zeta_urdf_description/meshes/FL_2_Motor_1.stl" scale="0.001 0.001 0.001"/>
@@ -334,5 +286,5 @@
   </visual>
   <collision>
-    <origin xyz="-0.721623 0.364211 -0.190939" rpy="0 0 0"/>
+    <origin xyz="-0.12822 -0.120819 -0.154456" rpy="0 0 0"/>
     <geometry>
       <mesh filename="package://zeta_urdf_description/meshes/FL_2_Motor_1.stl" scale="0.001 0.001 0.001"/>
@@ -342,13 +294,10 @@
 <link name="FL_1_Motor_1">
   <inertial>
-    <origin xyz="0.0027442419607356383 -0.00023296830563640514 0.00274502873903551" rpy="0 0 0"/>
+    <origin xyz="0.002744092080384855 -0.00023292577938141545 0.0027444919831759312" rpy="0 0 0"/>
     <mass value="0.09250068837133453"/>
-    <inertia ixx="0.0001" ixy="0.000"  ixz="0.000"
-         iyy="0.0001" iyz="0.000"
-         izz="0.0001"
-/>
-  </inertial>
-  <visual>
-    <origin xyz="-0.673893 0.379461 -0.143209" rpy="0 0 0"/>
+    <inertia ixx="1.8e-05" iyy="2e-05" izz="1.8e-05" ixy="-0.0" iyz="-0.0" ixz="-5e-06"/>
+  </inertial>
+  <visual>
+    <origin xyz="-0.08049 -0.105569 -0.106726" rpy="0 0 0"/>
     <geometry>
       <mesh filename="package://zeta_urdf_description/meshes/FL_1_Motor_1.stl" scale="0.001 0.001 0.001"/>
@@ -357,5 +306,5 @@
   </visual>
   <collision>
-    <origin xyz="-0.673893 0.379461 -0.143209" rpy="0 0 0"/>
+    <origin xyz="-0.08049 -0.105569 -0.106726" rpy="0 0 0"/>
     <geometry>
       <mesh filename="package://zeta_urdf_description/meshes/FL_1_Motor_1.stl" scale="0.001 0.001 0.001"/>
@@ -365,13 +314,10 @@
 <link name="FL_3_Motor_1">
   <inertial>
-    <origin xyz="0.00023268298076506433 -0.0038812370107810246 -4.0692889374804864e-07" rpy="0 0 0"/>
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